Commit message: urdf updates lite6

File: src/curobo/content/assets/robot/lite6/lite6.urdf (robot description, URDF)
Before this commit: robot lite6, 19 links, 18 joints
Links:
- link link_eef: geometry collision mesh filename=package://xarm_description/meshes/camera/realsense/collisio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; visual mesh filename=package://xarm_description/meshes/camera/realsense/visual/d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

Commit message: lite6 with gripper and camera update

File: src/curobo/content/assets/robot/lite6/lite6.urdf (robot description, URDF)
Before this commit: robot lite6, 19 links, 18 joints
Links:
- link link_eef: geometry collision mesh filename=meshes/collision/d435_with_cam_stand.stl; visual mesh filename=meshes/visual/d435_with_cam_stand.stl
- link uflite_gripper_link: geometry collision mesh filename=meshes/collision/gripper_lite.stl; visual mesh filename=meshes/visual/gripper_lite.stl
