Commit message: xarm7 updates

File: src/curobo/content/assets/robot/xarm7/xarm7.urdf (robot description, URDF)
Before this commit: robot xarm7, 26 links, 25 joints
Links:
- link left_finger: geometry collision mesh filename=meshes/visual/left_finger.stl; visual mesh filename=meshes/visual/left_finger.stl
- link left_inner_knuckle: geometry collision mesh filename=meshes/visual/left_inner_knuckle.stl; visual mesh filename=meshes/visual/left_inner_knuckle.stl
- link left_outer_knuckle: geometry collision mesh filename=meshes/visual/left_outer_knuckle.stl; visual mesh filename=meshes/visual/left_outer_knuckle.stl
- link link1: geometry collision mesh filename=meshes/visual/link1.stl; visual mesh filename=meshes/visual/link1.stl
- link link2: geometry collision mesh filename=meshes/visual/link2.stl; visual mesh filename=meshes/visual/link2.stl
- link link3: geometry collision mesh filename=meshes/visual/link3.stl; visual mesh filename=meshes/visual/link3.stl
- link link4: geometry collision mesh filename=meshes/visual/link4.stl; visual mesh filename=meshes/visual/link4.stl
- link link5: geometry collision mesh filename=meshes/visual/link5.stl; visual mesh filename=meshes/visual/link5.stl
- link link6: geometry collision mesh filename=meshes/visual/link6.stl; visual mesh filename=meshes/visual/link6.stl
- link link7: geometry collision mesh filename=meshes/visual/end_tool.stl; visual mesh filename=meshes/visual/link7.stl
- link link_base: geometry collision mesh filename=meshes/visual/link_base.stl; visual mesh filename=meshes/visual/link_base.stl
- link link_eef: geometry collision mesh filename=meshes/visual/d435_with_cam_stand.stl; visual mesh filename=meshes/visual/d435_with_cam_stand.stl
- link right_finger: geometry collision mesh filename=meshes/visual/right_finger.stl; visual mesh filename=meshes/visual/right_finger.stl
- link right_inner_knuckle: geometry collision mesh filename=meshes/visual/right_inner_knuckle.stl; visual mesh filename=meshes/visual/right_inner_knuckle.stl
- link right_outer_knuckle: geometry collision mesh filename=meshes/visual/right_outer_knuckle.stl; visual mesh filename=meshes/visual/right_outer_knuckle.stl
- link xarm_gripper_base_link: geometry collision mesh filename=meshes/visual/gripper_base_link.stl; visual mesh filename=meshes/visual/gripper_base_link.stl
